Commit message: Added gripper controller

File: src/so101_description/urdf/so101.ros2_control.xacro (robot description, xacro)
@@ -34,4 +34,9 @@
                 <state_interface name="velocity" />
             </joint>
+            <joint name="gripper">
+                <command_interface name="position" />
+                <state_interface name="position" />
+                <state_interface name="velocity" />
+            </joint>
         </ros2_control>
     </xacro:macro>

File: src/so101_description/urdf/so101.urdf.xacro (robot description, xacro)
@@ -310,5 +310,5 @@
     <child link="gripper_link" />
     <axis xyz="0 0 1" />
-    <limit effort="10" velocity="10" lower="-2.74385" upper="2.84121" />
+    <limit effort="10" velocity="10" lower="-2.7438473" upper="2.7438473" />
   </joint>
   <joint name="wrist_flex" type="revolute">

Commit message: Add real Feetech hardware backend for SO-101
- Parameterize the ros2_control xacro with hardware_type (mujoco|real),
  usb_port and joint_config_file; real uses FeetechHardwareInterface
  with servo IDs 1..6
- Add so101_bringup hardware.launch.py to start the real arm and its
  controllers
- Add use_sim_time launch argument to moveit.launch.py (default true)
- Document real robot usage in the README

File: src/so101_description/urdf/so101.ros2_control.xacro (robot description, xacro)
@@ -1,13 +1,24 @@
 <?xml version="1.0"?>
 <robot xmlns:xacro="http://www.ros.org/wiki/xacro">
-    <xacro:macro name="so101_ros2_control">
+    <xacro:macro name="so101_ros2_control" params="hardware_type usb_port joint_config_file">
+        <xacro:property name="is_real" value="${hardware_type == 'real'}" />
         <ros2_control name="SO101System" type="system">
             <hardware>
-                <plugin>mujoco_ros2_control/MujocoSystemInterface</plugin>
-                <param name="mujoco_model">
+                <xacro:if value="${hardware_type == 'mujoco'}">
+                    <plugin>mujoco_ros2_control/MujocoSystemInterface</plugin>
+                    <param name="mujoco_model">
                     $(find so101_description)/mujoco/scene.xml
                 </param>
+                </xacro:if>
+                <xacro:if value="${is_real}">
+                    <plugin>feetech_ros2_driver/FeetechHardwareInterface</plugin>
+                    <param name="usb_port">${usb_port}</param>
+                    <xacro:if value="${joint_config_file != ''}">
+                        <param name="joint_config_file">${joint_config_file}</param>
+                    </xacro:if>
+                </xacro:if>
             </hardware>
             <joint name="shoulder_pan">
+                <xacro:if value="${is_real}"><param name="id">1</param></xacro:if>
                 <command_interface name="position" />
                 <state_interface name="position" />
@@ -15,4 +26,5 @@
             </joint>
             <joint name="shoulder_lift">
+                <xacro:if value="${is_real}"><param name="id">2</param></xacro:if>
                 <command_interface name="position" />
                 <state_interface name="position" />
@@ -20,4 +32,5 @@
             </joint>
             <joint name="elbow_flex">
+                <xacro:if value="${is_real}"><param name="id">3</param></xacro:if>
                 <command_interface name="position" />
                 <state_interface name="position" />
@@ -25,4 +38,5 @@
             </joint>
             <joint name="wrist_flex">
+                <xacro:if value="${is_real}"><param name="id">4</param></xacro:if>
                 <command_interface name="position" />
                 <state_interface name="position" />
@@ -30,4 +44,5 @@
             </joint>
             <joint name="wrist_roll">
+                <xacro:if value="${is_real}"><param name="id">5</param></xacro:if>
                 <command_interface name="position" />
                 <state_interface name="position" />
@@ -35,4 +50,5 @@
             </joint>
             <joint name="gripper">
+                <xacro:if value="${is_real}"><param name="id">6</param></xacro:if>
                 <command_interface name="position" />
                 <state_interface name="position" />

File: src/so101_description/urdf/so101.urdf.xacro (robot description, xacro)
@@ -1,4 +1,7 @@
 <?xml version='1.0' encoding='utf-8'?>
 <robot name="so101" xmlns:xacro="http://www.ros.org/wiki/xacro">
+  <xacro:arg name="hardware_type" default="mujoco" />
+  <xacro:arg name="usb_port" default="/dev/ttyUSB0" />
+  <xacro:arg name="joint_config_file" default="" />
   <material name="3d_printed">
     <color rgba="1.0 0.82 0.12 1.0" />
@@ -341,4 +344,7 @@
   </joint>
   <xacro:include filename="$(find so101_description)/urdf/so101.ros2_control.xacro" />
-  <xacro:so101_ros2_control />
+  <xacro:so101_ros2_control
+    hardware_type="$(arg hardware_type)"
+    usb_port="$(arg usb_port)"
+    joint_config_file="$(arg joint_config_file)" />
 </robot>
