Commit message: Format so101.urdf.xacro

File: src/so101_description/urdf/so101.urdf.xacro (robot description, xacro)
@@ -11,5 +11,6 @@
       <origin xyz="0.0137179 -5.19711e-05 0.0334843" rpy="0 0 0" />
       <mass value="0.147" />
-      <inertia ixx="0.000114686" ixy="-4.59787e-07" ixz="4.97151e-06" iyy="0.000136117" iyz="9.75275e-08" izz="0.000130364" />
+      <inertia ixx="0.000114686" ixy="-4.59787e-07" ixz="4.97151e-06" iyy="0.000136117"
+        iyz="9.75275e-08" izz="0.000130364" />
     </inertial>
     <visual>
@@ -46,5 +47,6 @@
       <origin xyz="-0.0307604 -1.66727e-05 -0.0252713" rpy="0 0 0" />
       <mass value="0.100006" />
-      <inertia ixx="8.3759e-05" ixy="7.55525e-08" ixz="-1.16342e-06" iyy="8.10403e-05" iyz="1.54663e-07" izz="2.39783e-05" />
+      <inertia ixx="8.3759e-05" ixy="7.55525e-08" ixz="-1.16342e-06" iyy="8.10403e-05"
+        iyz="1.54663e-07" izz="2.39783e-05" />
     </inertial>
     <visual>
@@ -74,5 +76,6 @@
       <origin xyz="-0.0898471 -0.00838224 0.0184089" rpy="0 0 0" />
       <mass value="0.103" />
-      <inertia ixx="4.08002e-05" ixy="-1.97819e-05" ixz="-4.03016e-08" iyy="0.000147318" iyz="8.97326e-09" izz="0.000142487" />
+      <inertia ixx="4.08002e-05" ixy="-1.97819e-05" ixz="-4.03016e-08" iyy="0.000147318"
+        iyz="8.97326e-09" izz="0.000142487" />
     </inertial>
     <visual>
@@ -95,5 +98,6 @@
       <origin xyz="-0.0980701 0.00324376 0.0182831" rpy="0 0 0" />
       <mass value="0.104" />
-      <inertia ixx="2.87438e-05" ixy="7.41152e-06" ixz="1.26409e-06" iyy="0.000159844" iyz="-4.90188e-08" izz="0.00014529" />
+      <inertia ixx="2.87438e-05" ixy="7.41152e-06" ixz="1.26409e-06" iyy="0.000159844"
+        iyz="-4.90188e-08" izz="0.00014529" />
     </inertial>
     <visual>
@@ -123,5 +127,6 @@
       <origin xyz="-0.000103312 -0.0386143 0.0281156" rpy="0 0 0" />
       <mass value="0.079" />
-      <inertia ixx="3.68263e-05" ixy="1.7893e-08" ixz="-5.28128e-08" iyy="2.5391e-05" iyz="3.6412e-06" izz="2.1e-05" />
+      <inertia ixx="3.68263e-05" ixy="1.7893e-08" ixz="-5.28128e-08" iyy="2.5391e-05"
+        iyz="3.6412e-06" izz="2.1e-05" />
     </inertial>
     <visual>
@@ -144,5 +149,6 @@
       <origin xyz="0.000213627 0.000245138 -0.025187" rpy="0 0 0" />
       <mass value="0.087" />
-      <inertia ixx="2.75087e-05" ixy="-3.35241e-07" ixz="-5.7352e-06" iyy="4.33657e-05" iyz="-5.17847e-08" izz="3.45059e-05" />
+      <inertia ixx="2.75087e-05" ixy="-3.35241e-07" ixz="-5.7352e-06" iyy="4.33657e-05"
+        iyz="-5.17847e-08" izz="3.45059e-05" />
     </inertial>
     <visual>
@@ -179,5 +185,6 @@
       <origin xyz="-0.00157495 -0.0300244 0.0192755" rpy="0 0 0" />
       <mass value="0.012" />
-      <inertia ixx="6.61427e-06" ixy="-3.19807e-07" ixz="-5.90717e-09" iyy="1.89032e-06" iyz="-1.09945e-07" izz="5.28738e-06" />
+      <inertia ixx="6.61427e-06" ixy="-3.19807e-07" ixz="-5.90717e-09" iyy="1.89032e-06"
+        iyz="-1.09945e-07" izz="5.28738e-06" />
     </inertial>
     <visual>
@@ -231,3 +238,5 @@
     <limit effort="10" velocity="10" lower="-1.91986" upper="1.91986" />
   </joint>
+  <xacro:include filename="$(find so101_description)/urdf/so101.ros2_control.xacro" />
+  <xacro:so101_ros2_control />
 </robot>

Commit message: Add working MoveIt planning and MuJoCo execution

File: src/so101_description/urdf/so101.urdf.xacro (robot description, xacro)
@@ -21,4 +21,10 @@
       <material name="3d_printed" />
     </visual>
+    <collision>
+      <origin xyz="-0.00636471 -9.94414e-05 -0.0024" rpy="1.5708 -1.67685e-15 1.5708" />
+      <geometry>
+        <mesh filename="package://so101_description/meshes/base_motor_holder_so101_v1.stl" />
+      </geometry>
+    </collision>
     <visual>
       <origin xyz="-0.00636471 -8.97657e-09 -0.0024" rpy="1.5708 -2.78073e-29 1.5708" />
@@ -28,4 +34,10 @@
       <material name="3d_printed" />
     </visual>
+    <collision>
+      <origin xyz="-0.00636471 -8.97657e-09 -0.0024" rpy="1.5708 -2.78073e-29 1.5708" />
+      <geometry>
+        <mesh filename="package://so101_description/meshes/base_so101_v2.stl" />
+      </geometry>
+    </collision>
     <visual>
       <origin xyz="0.0263353 -8.97657e-09 0.0437" rpy="-8.21148e-16 7.84513e-18 1.249e-15" />
@@ -35,4 +47,10 @@
       <material name="sts3215" />
     </visual>
+    <collision>
+      <origin xyz="0.0263353 -8.97657e-09 0.0437" rpy="-8.21148e-16 7.84513e-18 1.249e-15" />
+      <geometry>
+        <mesh filename="package://so101_description/meshes/sts3215_03a_v1.stl" />
+      </geometry>
+    </collision>
     <visual>
       <origin xyz="-0.0309827 -0.000199441 0.0474" rpy="1.5708 -1.35493e-14 1.5708" />
@@ -42,4 +60,10 @@
       <material name="3d_printed" />
     </visual>
+    <collision>
+      <origin xyz="-0.0309827 -0.000199441 0.0474" rpy="1.5708 -1.35493e-14 1.5708" />
+      <geometry>
+        <mesh filename="package://so101_description/meshes/waveshare_mounting_plate_so101_v2.stl" />
+      </geometry>
+    </collision>
   </link>
   <link name="shoulder_link">
@@ -57,4 +81,10 @@
       <material name="sts3215" />
     </visual>
+    <collision>
+      <origin xyz="-0.0303992 0.000422241 -0.0417" rpy="1.5708 1.5708 0" />
+      <geometry>
+        <mesh filename="package://so101_description/meshes/sts3215_03a_v1.stl" />
+      </geometry>
+    </collision>
     <visual>
       <origin xyz="-0.0675992 -0.000177759 0.0158499" rpy="1.5708 -1.5708 0" />
@@ -64,4 +94,10 @@
       <material name="3d_printed" />
     </visual>
+    <collision>
+      <origin xyz="-0.0675992 -0.000177759 0.0158499" rpy="1.5708 -1.5708 0" />
+      <geometry>
+        <mesh filename="package://so101_description/meshes/motor_holder_so101_base_v1.stl" />
+      </geometry>
+    </collision>
     <visual>
       <origin xyz="0.0122008 2.22413e-05 0.0464" rpy="-1.5708 2.35221e-33 0" />
@@ -71,4 +107,10 @@
       <material name="3d_printed" />
     </visual>
+    <collision>
+      <origin xyz="0.0122008 2.22413e-05 0.0464" rpy="-1.5708 2.35221e-33 0" />
+      <geometry>
+        <mesh filename="package://so101_description/meshes/rotation_pitch_so101_v1.stl" />
+      </geometry>
+    </collision>
   </link>
   <link name="upper_arm_link">
@@ -86,4 +128,10 @@
       <material name="sts3215" />
     </visual>
+    <collision>
+      <origin xyz="-0.11257 -0.0155 0.0187" rpy="-3.14159 -5.27356e-16 -1.5708" />
+      <geometry>
+        <mesh filename="package://so101_description/meshes/sts3215_03a_v1.stl" />
+      </geometry>
+    </collision>
     <visual>
       <origin xyz="-0.065085 0.012 0.0182" rpy="3.14159 -0 -1.30911e-30" />
@@ -93,4 +141,10 @@
       <material name="3d_printed" />
     </visual>
+    <collision>
+      <origin xyz="-0.065085 0.012 0.0182" rpy="3.14159 -0 -1.30911e-30" />
+      <geometry>
+        <mesh filename="package://so101_description/meshes/upper_arm_so101_v1.stl" />
+      </geometry>
+    </collision>
   </link>
   <link name="lower_arm_link">
@@ -108,4 +162,10 @@
       <material name="3d_printed" />
     </visual>
+    <collision>
+      <origin xyz="-0.0648499 -0.032 0.0182" rpy="3.14159 -0 6.67202e-31" />
+      <geometry>
+        <mesh filename="package://so101_description/meshes/under_arm_so101_v1.stl" />
+      </geometry>
+    </collision>
     <visual>
       <origin xyz="-0.0648499 -0.032 0.018" rpy="-3.14159 -2.55351e-15 -1.83387e-30" />
@@ -115,4 +175,10 @@
       <material name="3d_printed" />
     </visual>
+    <collision>
+      <origin xyz="-0.0648499 -0.032 0.018" rpy="-3.14159 -2.55351e-15 -1.83387e-30" />
+      <geometry>
+        <mesh filename="package://so101_description/meshes/motor_holder_so101_wrist_v1.stl" />
+      </geometry>
+    </collision>
     <visual>
       <origin xyz="-0.1224 0.0052 0.0187" rpy="-3.14159 -7.88861e-31 -3.14159" />
@@ -122,4 +188,10 @@
       <material name="sts3215" />
     </visual>
+    <collision>
+      <origin xyz="-0.1224 0.0052 0.0187" rpy="-3.14159 -7.88861e-31 -3.14159" />
+      <geometry>
+        <mesh filename="package://so101_description/meshes/sts3215_03a_v1.stl" />
+      </geometry>
+    </collision>
   </link>
   <link name="wrist_link">
@@ -137,4 +209,10 @@
       <material name="sts3215" />
     </visual>
+    <collision>
+      <origin xyz="8.32667e-17 -0.0424 0.0306" rpy="1.5708 1.5708 0" />
+      <geometry>
+        <mesh filename="package://so101_description/meshes/sts3215_03a_no_horn_v1.stl" />
+      </geometry>
+    </collision>
     <visual>
       <origin xyz="0 -0.028 0.0181" rpy="-1.5708 -1.5708 0" />
@@ -144,4 +222,10 @@
       <material name="3d_printed" />
     </visual>
+    <collision>
+      <origin xyz="0 -0.028 0.0181" rpy="-1.5708 -1.5708 0" />
+      <geometry>
+        <mesh filename="package://so101_description/meshes/wrist_roll_pitch_so101_v2.stl" />
+      </geometry>
+    </collision>
   </link>
   <link name="gripper_link">
@@ -159,4 +243,10 @@
       <material name="sts3215" />
     </visual>
+    <collision>
+      <origin xyz="0.0077 0.0001 -0.0234" rpy="-1.5708 -5.19179e-17 -1.66533e-16" />
+      <geometry>
+        <mesh filename="package://so101_description/meshes/sts3215_03a_v1.stl" />
+      </geometry>
+    </collision>
     <visual>
       <origin xyz="8.32667e-17 -0.000218214 0.000949706" rpy="-3.14159 -5.55112e-17 0" />
@@ -166,4 +256,10 @@
       <material name="3d_printed" />
     </visual>
+    <collision>
+      <origin xyz="8.32667e-17 -0.000218214 0.000949706" rpy="-3.14159 -5.55112e-17 0" />
+      <geometry>
+        <mesh filename="package://so101_description/meshes/wrist_roll_follower_so101_v1.stl" />
+      </geometry>
+    </collision>
   </link>
   <link name="gripper_frame_link">
@@ -195,4 +291,10 @@
       <material name="3d_printed" />
     </visual>
+    <collision>
+      <origin xyz="-5.55112e-17 -5.55112e-17 0.0189" rpy="9.53145e-17 6.93889e-18 1.24077e-24" />
+      <geometry>
+        <mesh filename="package://so101_description/meshes/moving_jaw_so101_v1.stl" />
+      </geometry>
+    </collision>
   </link>
   <joint name="gripper" type="revolute">

Commit message: Align MuJoCo gripper TCP with MoveIt frame

File: src/so101_description/urdf/so101.urdf.xacro (robot description, xacro)
@@ -272,5 +272,5 @@
   </link>
   <joint name="gripper_frame_joint" type="fixed">
-    <origin xyz="-0.0079 -0.000218121 -0.0981274" rpy="0 3.14159 0" />
+    <origin xyz="-0.0079 -0.000218121 -0.0981274" rpy="0 3.141592653589793 0" />
     <parent link="gripper_link" />
     <child link="gripper_frame_link" />

Commit message: Load follower calibration by default on the real arm
- Add scripts/generate_follower_joint_config.py to convert a LeRobot
  follower calibration JSON into so101_bringup/config/follower_joints.yaml
- Commit the follower arm's calibration and make it the default
  joint_config_file in hardware.launch.py
- Widen the shoulder_lift lower limit to -1.9 rad so the folded rest
  pose stays inside the URDF limit
- Add feetech_ros2_driver as a git submodule
- Document the calibration workflow in the README

File: src/so101_description/urdf/so101.urdf.xacro (robot description, xacro)
@@ -334,5 +334,6 @@
     <child link="upper_arm_link" />
     <axis xyz="0 0 1" />
-    <limit effort="10" velocity="10" lower="-1.74533" upper="1.74533" />
+    <!-- Lower bound covers the folded rest pose on the real arm (calibrated range_min ~ -1.896 rad) -->
+    <limit effort="10" velocity="10" lower="-1.9" upper="1.74533" />
   </joint>
   <joint name="shoulder_pan" type="revolute">
